File: USBCEXPERIMENT/USBCEXPERIMENT.sch (KiCad schematic (older format))
At the start: 3 parts, among them J1 USB_C_Receptacle, J2 Conn_01x10_Male, J3 Conn_01x10_Male

Commit message: started to add a simple version to the PCB
Parts:
- added J4: USB_C_Receptacle, footprint:usb-c-pcb, symbol Connector:USB_C_Receptacle
- added J5: Conn_01x10_Male, Connector_PinHeader_2.54mm:PinHeader_1x10_P2.54mm_Vertical, symbol Connector:Conn_01x10_Male
Connections:
- wire segments 62 -> 104
